File: pcb/Project_Main_V1/SOC.kicad_sch (KiCad schematic)
At the start: 1 part, among them IC1 XC7Z007S-1CLG225C

Commit message: Updated Schematics and Footprints of SOC
Updated Schematics and Footprints of SOC. The pitch is actually 0.8mm
Parts:
- removed IC1: XC7Z007S-1CLG225C, XC7Z007S_1CLG225C:BGA225C80P15X15_1300X1300X150, symbol XC7Z007S-1CLG225C:XC7Z007S-1CLG225C
- added U1: XC7Z010-1CLG400C, footprints:CLG400_AMD, symbol 2024-09-09_01-22-32:XC7Z010-1CLG400C
